Commit message: update collision geometry to match new urdf

File: urdf/za.urdf (robot description, URDF)
Before this commit: robot za, 11 links, 10 joints
Links:
- link base_link: geometry collision mesh filename=package://za_description/meshes/base_link_collision.stl; visual mesh filename=package://za_description/meshes/base_link.dae
- link link_1: geometry collision mesh filename=package://za_description/meshes/link_1_collision.stl; visual mesh filename=package://za_description/meshes/link_1.dae
- link link_2: geometry collision mesh filename=package://za_description/meshes/link_2_collision.stl; visual mesh filename=package://za_description/meshes/link_2.dae
- link link_3: geometry collision mesh filename=package://za_description/meshes/link_3_collision.stl; visual mesh filename=package://za_description/meshes/link_3.dae
- link link_4: geometry collision mesh filename=package://za_description/meshes/link_4_collision.stl; visual mesh filename=package://za_description/meshes/link_4.dae
- link link_5: geometry collision mesh filename=package://za_description/meshes/link_5_collision.stl; visual mesh filename=package://za_description/meshes/link_5.dae
- link link_6: geometry collision mesh filename=package://za_description/meshes/link_6_collision.stl; visual mesh filename=package://za_description/meshes/link_6.dae
Joints:
- joint joint_1: origin xyz=0 0 0.279 rpy=0.0 0.0 0.0 -> xyz=0 0 0.45 rpy=0.0 0.0 0.0
- joint joint_2: origin xyz=0.025 0 0.171 rpy=0.0 0.0 0.0 -> xyz=0.025 0 0.0 rpy=0.0 0.0 0.0
- joint joint_3: origin xyz=0.0 -0.001 0.454 rpy=0.0 1.5707963267948966 0.0 -> xyz=0.0 0.0 0.454 rpy=0.0 0.0 0.0
- joint joint_4: axis 0 0 1 -> 1 0 0; origin xyz=-0.035 -0 0.123 rpy=0.0 0.0 0.0 -> xyz=0.0 0.0 0.035 rpy=0.0 0.0 0.0
- joint joint_5: origin xyz=0.0 0.001 0.2965 rpy=0.0 0.0 0.0 -> xyz=0.4195 0.00 0.0 rpy=0.0 0.0 0.0
- joint joint_6: axis 0 0 1 -> 1 0 0; origin xyz=0 0 0.1 rpy=0.0 0.0 0.0 -> xyz=0.1 0.0 0.0 rpy=0.0 0.0 0.0

File: urdf/za_macro.xacro (robot description, xacro)
@@ -6,13 +6,11 @@
       <visual>
         <geometry>
-          <mesh filename="package://za_description/meshes/base_link.dae"/>
+          <mesh filename="package://za_description/meshes/visual/base_link.dae"/>
         </geometry>
-        <origin rpy="0.0 0 0.0" xyz="0 0 0"/>
       </visual>
       <collision>
         <geometry>
-          <mesh filename="package://za_description/meshes/base_link_collision.stl"/>
+          <mesh filename="package://za_description/meshes/collision/base_link_collision.stl"/>
         </geometry>
-        <origin rpy="0.0 0 0.0" xyz="0 0 0"/>
       </collision>
     </link>
@@ -20,12 +18,11 @@
       <visual>
         <geometry>
-          <mesh filename="package://za_description/meshes/link_1.dae"/>
+          <mesh filename="package://za_description/meshes/visual/link_1.dae"/>
         </geometry>
       </visual>
       <collision>
         <geometry>
-          <mesh filename="package://za_description/meshes/link_1_collision.stl"/>
+          <mesh filename="package://za_description/meshes/collision/link_1_collision.stl"/>
         </geometry>
-        <origin rpy="0.0 0 0.0" xyz="0 0 0"/>
       </collision>
       <inertial>
@@ -37,13 +34,11 @@
       <visual>
         <geometry>
-          <mesh filename="package://za_description/meshes/link_2.dae"/>
+          <mesh filename="package://za_description/meshes/visual/link_2.dae"/>
         </geometry>
-        <origin rpy="0.0 0 0.0" xyz="0 0 0"/>
       </visual>
       <collision>
         <geometry>
-          <mesh filename="package://za_description/meshes/link_2_collision.stl"/>
+          <mesh filename="package://za_description/meshes/collision/link_2_collision.stl"/>
         </geometry>
-        <origin rpy="0.0 0 0.0" xyz="0 0 0"/>
       </collision>
       <inertial>
@@ -55,13 +50,11 @@
       <visual>
         <geometry>
-          <mesh filename="package://za_description/meshes/link_3.dae"/>
+          <mesh filename="package://za_description/meshes/visual/link_3.dae"/>
         </geometry>
-        <origin rpy="0.0 0 0.0" xyz="0 0 0"/>
       </visual>
       <collision>
         <geometry>
-          <mesh filename="package://za_description/meshes/link_3_collision.stl"/>
+          <mesh filename="package://za_description/meshes/collision/link_3_collision.stl"/>
         </geometry>
-        <origin rpy="0.0 0 0.0" xyz="-0 0 0"/>
       </collision>
       <inertial>
@@ -73,13 +66,11 @@
       <visual>
         <geometry>
-          <mesh filename="package://za_description/meshes/link_4.dae"/>
+          <mesh filename="package://za_description/meshes/visual/link_4.dae"/>
         </geometry>
-        <origin rpy="0.0 0.0 0.0" xyz="0 0 0"/>
       </visual>
       <collision>
         <geometry>
-          <mesh filename="package://za_description/meshes/link_4_collision.stl"/>
+          <mesh filename="package://za_description/meshes/collision/link_4_collision.stl"/>
         </geometry>
-        <origin rpy="0.0 0 0.0" xyz="0 0 0"/>
       </collision>
       <inertial>
@@ -91,13 +82,11 @@
       <visual>
         <geometry>
-          <mesh filename="package://za_description/meshes/link_5.dae"/>
+          <mesh filename="package://za_description/meshes/visual/link_5.dae"/>
         </geometry>
-        <origin rpy="0 0 0" xyz="0 0 0"/>
       </visual>
       <collision>
         <geometry>
-          <mesh filename="package://za_description/meshes/link_5_collision.stl"/>
+          <mesh filename="package://za_description/meshes/collision/link_5_collision.stl"/>
         </geometry>
-        <origin rpy="0 0 0" xyz="0 0 0"/>
       </collision>
       <inertial>
@@ -109,13 +98,11 @@
       <visual>
         <geometry>
-          <mesh filename="package://za_description/meshes/link_6.dae"/>
+          <mesh filename="package://za_description/meshes/visual/link_6.dae"/>
         </geometry>
-        <origin rpy="0 0 0.0" xyz="0 0 0"/>
       </visual>
       <collision>
         <geometry>
-          <mesh filename="package://za_description/meshes/link_6_collision.stl"/>
+          <mesh filename="package://za_description/meshes/collision/link_6_collision.stl"/>
         </geometry>
-        <origin rpy="0 0 0.0" xyz="0 0 0"/>
       </collision>
       <inertial>
@@ -126,44 +113,44 @@
     <!-- joint list -->
     <joint name="${prefix}joint_1" type="revolute">
-      <limit effort="1000.0" lower="-2.96" upper="2.96" velocity="2.6"/>
+      <origin rpy="0.0 0.0 0.0" xyz="0 0 0.45"/>
+      <axis xyz="0 0 1"/>
       <parent link="${prefix}base_link"/>
       <child link="${prefix}link_1"/>
-      <axis xyz="0 0 1"/>
-      <origin rpy="0.0 0.0 0.0" xyz="0 0 0.279"/>
+      <limit effort="1000.0" lower="-2.96" upper="2.96" velocity="2.6"/>
     </joint>
     <joint name="${prefix}joint_2" type="revolute">
-      <limit effort="1000.0" lower="-1.74" upper="2.35" velocity="1.9"/>
+      <origin rpy="0.0 0.0 0.0" xyz="0.025 0 0.0"/>
+      <axis xyz="0 1 0"/>
       <parent link="${prefix}link_1"/>
       <child link="${prefix}link_2"/>
-      <axis xyz="0 1 0"/>
-      <origin rpy="0.0 0.0 0.0" xyz="0.025 0 0.171"/>
+      <limit effort="1000.0" lower="-1.74" upper="2.35" velocity="1.9"/>
     </joint>
     <joint name="${prefix}joint_3" type="revolute">
-      <limit effort="1000.0" lower="-1.570796" upper="1.15" velocity="2.6"/>
+      <origin rpy="0.0 0.0 0.0" xyz="0.0 0.0 0.454"/>
+      <axis xyz="0 1 0"/>
       <parent link="${prefix}link_2"/>
       <child link="${prefix}link_3"/>
-      <axis xyz="0 1 0"/>
-      <origin rpy="0.0 ${pi/2.0} 0.0" xyz="0.0 -0.001 0.454"/>
+      <limit effort="1000.0" lower="-1.570796" upper="1.15" velocity="2.6"/>
     </joint>
     <joint name="${prefix}joint_4" type="revolute">
-      <limit effort="1000.0" lower="-2.6" upper="2.6" velocity="3.5"/>
+      <origin rpy="0.0 0.0 0.0" xyz="0.0 0.0 0.035"/>
+      <axis xyz="1 0 0"/>
       <parent link="${prefix}link_3"/>
       <child link="${prefix}link_4"/>
-      <axis xyz="0 0 1"/>
-      <origin rpy="0.0 0.0 0.0" xyz="-0.035 -0 0.123"/>
+      <limit effort="1000.0" lower="-2.6" upper="2.6" velocity="3.5"/>
     </joint>
     <joint name="${prefix}joint_5" type="revolute">
-      <limit effort="1000.0" lower="-2.49" upper="2.49" velocity="3.9"/>
+      <origin rpy="0.0 0.0 0.0" xyz="0.4195 0.0 0.0"/>
+      <axis xyz="0 1 0"/>
       <parent link="${prefix}link_4"/>
       <child link="${prefix}link_5"/>
-      <axis xyz="0 1 0"/>
-      <origin rpy="0.0 0.0 0.0" xyz="0.0 0.001 0.2965"/>
+      <limit effort="1000.0" lower="-2.49" upper="2.49" velocity="3.9"/>
     </joint>
     <joint name="${prefix}joint_6" type="revolute">
-      <limit effort="1000.0" lower="${pi*-1}" upper="${pi*1}" velocity="${pi*2}"/>
+      <origin rpy="0.0 0.0 0.0" xyz="0.1 0.0 0.0"/>
+      <axis xyz="1 0 0"/>
       <parent link="${prefix}link_5"/>
       <child link="${prefix}link_6"/>
-      <axis xyz="0 0 1"/>
-      <origin rpy="0.0 0.0 0.0" xyz="0 0 0.1"/>
+      <limit effort="1000.0" lower="${pi*-1}" upper="${pi*1}" velocity="${pi*2}"/>
     </joint>
     <!-- ROS-Industrial 'base' frame: base_link to Fanuc World Coordinates transform -->
@@ -188,5 +175,5 @@
         <!-- marker -->
         <origin xyz="${tool0_trans}" rpy="${tool0_rot}" />
-        <parent link="${prefix}link_6" />
+        <parent link="${prefix}flange" />
         <child link="${prefix}tool0" />
       </joint>
@@ -195,5 +182,5 @@
       <joint name="${prefix}link_6_tool0" type="floating">
         <origin xyz="0 0 0" rpy="0 0 0" />
-        <parent link="${prefix}link_6" />
+        <parent link="${prefix}flange" />
         <child link="${prefix}tool0" />
       </joint>
