Commit message: update inertia values with solidworks data

File: urdf/utils.xacro (robot description, xacro)
@@ -54,5 +54,5 @@
   <!-- ============================================================ -->
   <xacro:macro name="transmission-za-model" params="arm_id root tip">
-    <transmission name="${arm_id}_za_model">
+    <transmission name="${arm_id}za_model">
       <type>za_hw/ZaModelInterface</type>
       <joint name="${root}">

File: urdf/za_macro.xacro (robot description, xacro)
@@ -18,7 +18,7 @@
       </collision>
       <inertial>
-        <origin xyz="-0.01236763 -0.00120116 0.13466856"/>
-        <mass value="18.32700000"/>
-        <inertia ixx="0.16366788" ixy="-0.00000166" ixz="-0.00348810" iyy="0.22044850" iyz="0.00000286" izz="0.17770306"/>
+        <origin xyz="-0.035356 -0.000003 0.142049"/>
+        <mass value="18.327"/>
+        <inertia ixx="0.185203" ixy="0.000006" ixz="0.016506" iyy="0.232301" iyz="0.000014" izz="0.163415"/>
       </inertial>
     </link>
@@ -35,7 +35,7 @@
       </collision>
       <inertial>
-        <origin xyz="0.01021395 0.00697465 -0.07935107"/>
-        <mass value="13.44000000"/>
-        <inertia ixx="0.13591253" ixy="0.00009739" ixz="-0.00604284" iyy="0.11223931" iyz="0.00027520" izz="0.10172556"/>
+        <origin xyz="0.009612 0.016390 -0.065742"/>
+        <mass value="13.44"/>
+        <inertia ixx="0.178493" ixy="0.002772" ixz="0.010363" iyy="0.126756" iyz="0.016161" izz="0.130031"/>
       </inertial>
     </link>
@@ -52,7 +52,7 @@
       </collision>
       <inertial>
-        <origin xyz="-0.00387549 -0.00718854 0.27138897"/>
-        <mass value="17.11000000"/>
-        <inertia ixx="0.52527032" ixy="0.00015072" ixz="0.00040686" iyy="0.50042448" iyz="0.00016892" izz="0.09140527"/>
+        <origin xyz="-0.003803 0.001296 0.191397"/>
+        <mass value="17.11"/>
+        <inertia ixx="0.740919" ixy="-0.003160" ixz="-0.003160" iyy="0.699365" iyz="0.039435" izz="0.100361"/>
       </inertial>
     </link>
@@ -69,7 +69,7 @@
       </collision>
       <inertial>
-        <origin xyz="0.02825936 0.00083544 -0.00574226"/>
-        <mass value="7.33000000"/>
-        <inertia ixx="0.02513174" ixy="0.00012221" ixz="-0.00333856" iyy="0.03765338" iyz="-0.00009292" izz="0.02694824"/>
+        <origin xyz="0.019381 -0.007200 -0.002694"/>
+        <mass value="7.33"/>
+        <inertia ixx="0.027465" ixy="0.001126" ixz="0.004749" iyy="0.037555" iyz="-0.000148" izz="0.031377"/>
       </inertial>
     </link>
@@ -86,7 +86,7 @@
       </collision>
       <inertial>
-        <origin xyz="0.30544152 0.00346903 0.00392327"/>
-        <mass value="6.11000000"/>
-        <inertia ixx="0.01559502" ixy="-0.00031903" ixz="0.00008767" iyy="0.05602555" iyz="-0.00001324" izz="0.06119102"/>
+        <origin xyz="0.290062 0.005593 0.000640"/>
+        <mass value="6.11"/>
+        <inertia ixx="0.019909" ixy="0.003159" ixz="-0.000103" iyy="0.058941" iyz="-0.000022" izz="0.066959"/>
       </inertial>
     </link>
@@ -103,7 +103,7 @@
       </collision>
       <inertial>
-        <origin xyz="-0.00517740 0.00016151 0.00015567"/>
-        <mass value="2.44000000"/>
-        <inertia ixx="0.00267434" ixy="0.00000003" ixz="-0.00000009" iyy="0.00582935" iyz="-0.00000003" izz="0.00571470"/>
+        <origin xyz="0.009621 0.000953 0.000305"/>
+        <mass value="2.44"/>
+        <inertia ixx="0.002635" ixy="-0.000031" ixz="-0.000023" iyy="0.005551" iyz="0.000004" izz="0.005487"/>
       </inertial>
     </link>
@@ -120,7 +120,7 @@
       </collision>
       <inertial>
-        <origin xyz="-0.00968719 -0.00009104 0.00002796"/>
-        <mass value="0.24400000"/>
-        <inertia ixx="0.00010069" ixy="0.00000000" ixz="0.00000000" iyy="0.00006352" iyz="0.00000000" izz="0.00006352"/>
+        <origin xyz="-0.012049 0.000000 0.000000"/>
+        <mass value="0.244"/>
+        <inertia ixx="0.000106" ixy="0.000000" ixz="0.000000" iyy="0.000064" iyz="0.000000" izz="0.000064"/>
       </inertial>
     </link>

Commit message: add joint reductions and dynamics

File: urdf/utils.xacro (robot description, xacro)
@@ -10,5 +10,5 @@
     </inertial>
   </xacro:macro>
-  <xacro:macro name="gazebo-joint" params="joint transmission:=hardware_interface/EffortJointInterface">
+  <xacro:macro name="gazebo-joint" params="joint transmission:=hardware_interface/EffortJointInterface reduction:=1">
     <transmission name="${joint}_transmission">
       <type>transmission_interface/SimpleTransmission</type>
@@ -18,5 +18,5 @@
       <actuator name="${joint}_motor">
         <hardwareInterface>${transmission}</hardwareInterface>
-        <mechanicalReduction>1</mechanicalReduction>
+        <mechanicalReduction>${reduction}</mechanicalReduction>
       </actuator>
     </transmission>

File: urdf/za_macro.xacro (robot description, xacro)
@@ -132,6 +132,6 @@
       <child link="${prefix}link_1"/>
       <limit effort="1000.0" lower="-2.96" upper="2.96" velocity="2.6"/>
-      <dynamics damping="0.003" friction="0.0" mu_coulomb="0" mu_viscous="16" />
-    </joint>
+      <dynamics damping="0.003" friction="0.0"/>
+  </joint>
     <joint name="${prefix}joint_2" type="revolute">
       <origin rpy="0.0 0.0 0.0" xyz="0.025 0 0.0"/>
@@ -140,5 +140,5 @@
       <child link="${prefix}link_2"/>
       <limit effort="1000.0" lower="-1.74" upper="2.35" velocity="1.9"/>
-      <dynamics damping="0.003" friction="0.0" mu_coulomb="0" mu_viscous="16" />
+      <dynamics damping="0.003" friction="0.0"/>
     </joint>
     <joint name="${prefix}joint_3" type="revolute">
@@ -148,5 +148,5 @@
       <child link="${prefix}link_3"/>
       <limit effort="1000.0" lower="-1.570796" upper="1.15" velocity="2.6"/>
-      <dynamics damping="0.003" friction="0.0" mu_coulomb="0" mu_viscous="16" />
+      <dynamics damping="0.003" friction="0.0"/>
     </joint>
     <joint name="${prefix}joint_4" type="revolute">
@@ -156,5 +156,5 @@
       <child link="${prefix}link_4"/>
       <limit effort="1000.0" lower="-2.6" upper="2.6" velocity="3.5"/>
-      <dynamics damping="0.003" friction="0.0" mu_coulomb="0" mu_viscous="16" />
+      <dynamics damping="0.003" friction="0.0"/>
     </joint>
     <joint name="${prefix}joint_5" type="revolute">
@@ -164,5 +164,5 @@
       <child link="${prefix}link_5"/>
       <limit effort="1000.0" lower="-2.49" upper="2.49" velocity="3.9"/>
-      <dynamics damping="0.003" friction="0.0" mu_coulomb="0" mu_viscous="16" />
+      <dynamics damping="0.003" friction="0.0"/>
     </joint>
     <joint name="${prefix}joint_6" type="revolute">
@@ -172,5 +172,5 @@
       <child link="${prefix}link_6"/>
       <limit effort="1000.0" lower="${pi*-1}" upper="${pi*1}" velocity="${pi*2}"/>
-      <dynamics damping="0.003" friction="0.0" mu_coulomb="0" mu_viscous="16" />
+      <dynamics damping="0.003" friction="0.0"/>
     </joint>
     <!-- ROS-Industrial 'base' frame: base_link to Fanuc World Coordinates transform -->
@@ -198,22 +198,22 @@
     <!-- Define additional Gazebo tags -->
     <xacro:if value="$(arg gazebo)">
-      <xacro:gazebo-joint joint="${prefix}joint_1" transmission="hardware_interface/EffortJointInterface" />
-      <xacro:gazebo-joint joint="${prefix}joint_2" transmission="hardware_interface/EffortJointInterface" />
-      <xacro:gazebo-joint joint="${prefix}joint_3" transmission="hardware_interface/EffortJointInterface" />
-      <xacro:gazebo-joint joint="${prefix}joint_4" transmission="hardware_interface/EffortJointInterface" />
-      <xacro:gazebo-joint joint="${prefix}joint_5" transmission="hardware_interface/EffortJointInterface" />
-      <xacro:gazebo-joint joint="${prefix}joint_6" transmission="hardware_interface/EffortJointInterface" />
-      <xacro:gazebo-joint joint="${prefix}joint_1" transmission="hardware_interface/VelocityJointInterface" />
-      <xacro:gazebo-joint joint="${prefix}joint_2" transmission="hardware_interface/VelocityJointInterface" />
-      <xacro:gazebo-joint joint="${prefix}joint_3" transmission="hardware_interface/VelocityJointInterface" />
-      <xacro:gazebo-joint joint="${prefix}joint_4" transmission="hardware_interface/VelocityJointInterface" />
-      <xacro:gazebo-joint joint="${prefix}joint_5" transmission="hardware_interface/VelocityJointInterface" />
-      <xacro:gazebo-joint joint="${prefix}joint_6" transmission="hardware_interface/VelocityJointInterface" />
-      <xacro:gazebo-joint joint="${prefix}joint_1" transmission="hardware_interface/PositionJointInterface" />
-      <xacro:gazebo-joint joint="${prefix}joint_2" transmission="hardware_interface/PositionJointInterface" />
-      <xacro:gazebo-joint joint="${prefix}joint_3" transmission="hardware_interface/PositionJointInterface" />
-      <xacro:gazebo-joint joint="${prefix}joint_4" transmission="hardware_interface/PositionJointInterface" />
-      <xacro:gazebo-joint joint="${prefix}joint_5" transmission="hardware_interface/PositionJointInterface" />
-      <xacro:gazebo-joint joint="${prefix}joint_6" transmission="hardware_interface/PositionJointInterface" />
+      <xacro:gazebo-joint joint="${prefix}joint_1" transmission="hardware_interface/EffortJointInterface" reduction="1.5"/>
+      <xacro:gazebo-joint joint="${prefix}joint_2" transmission="hardware_interface/EffortJointInterface" reduction="100"/>
+      <xacro:gazebo-joint joint="${prefix}joint_3" transmission="hardware_interface/EffortJointInterface" reduction="50"/>
+      <xacro:gazebo-joint joint="${prefix}joint_4" transmission="hardware_interface/EffortJointInterface" reduction="1.25"/>
+      <xacro:gazebo-joint joint="${prefix}joint_5" transmission="hardware_interface/EffortJointInterface" reduction="50"/>
+      <xacro:gazebo-joint joint="${prefix}joint_6" transmission="hardware_interface/EffortJointInterface" reduction="30"/>
+      <xacro:gazebo-joint joint="${prefix}joint_1" transmission="hardware_interface/VelocityJointInterface" reduction="1.5"/>
+      <xacro:gazebo-joint joint="${prefix}joint_2" transmission="hardware_interface/VelocityJointInterface" reduction="100"/>
+      <xacro:gazebo-joint joint="${prefix}joint_3" transmission="hardware_interface/VelocityJointInterface" reduction="50"/>
+      <xacro:gazebo-joint joint="${prefix}joint_4" transmission="hardware_interface/VelocityJointInterface" reduction="1.25"/>
+      <xacro:gazebo-joint joint="${prefix}joint_5" transmission="hardware_interface/VelocityJointInterface" reduction="50"/>
+      <xacro:gazebo-joint joint="${prefix}joint_6" transmission="hardware_interface/VelocityJointInterface" reduction="30"/>
+      <xacro:gazebo-joint joint="${prefix}joint_1" transmission="hardware_interface/PositionJointInterface" reduction="1.5"/>
+      <xacro:gazebo-joint joint="${prefix}joint_2" transmission="hardware_interface/PositionJointInterface" reduction="100"/>
+      <xacro:gazebo-joint joint="${prefix}joint_3" transmission="hardware_interface/PositionJointInterface" reduction="50"/>
+      <xacro:gazebo-joint joint="${prefix}joint_4" transmission="hardware_interface/PositionJointInterface" reduction="1.25"/>
+      <xacro:gazebo-joint joint="${prefix}joint_5" transmission="hardware_interface/PositionJointInterface" reduction="50"/>
+      <xacro:gazebo-joint joint="${prefix}joint_6" transmission="hardware_interface/PositionJointInterface" reduction="30"/>
       <xacro:transmission-za-state arm_id="${prefix}" />
       <xacro:transmission-za-model arm_id="${prefix}"
