Commit message: add case for including urdf hardware

File: urdf/za.ros2_control.xacro (robot description, xacro)
@@ -1,8 +1,13 @@
 <?xml version="1.0"?>
 <robot xmlns:xacro="http://www.ros.org/wiki/xacro">
-  <xacro:macro name="za_ros2_control" params="prefix">
-    <ros2_control name="za_ros2_control" type="system">
+  <xacro:macro name="za_ros2_control" params="prefix use_mock_hardware:=^|true">
+    <ros2_control name="${prefix}ros2_control" type="system">
       <hardware>
-        <plugin>mock_components/GenericSystem</plugin>
+        <xacro:if value="${use_mock_hardware}">
+          <plugin>mock_components/GenericSystem</plugin>
+        </xacro:if>
+        <xacro:unless value="${use_mock_hardware}">
+          <!-- <plugin>hal_ros_control/HalHardware</plugin> -->
+        </xacro:unless>
       </hardware>
       <joint name="${prefix}joint_1">

File: urdf/za.xacro (robot description, xacro)
@@ -2,4 +2,6 @@
 <robot name="za" xmlns:xacro="http://www.ros.org/wiki/xacro">
   <xacro:arg name="prefix" default=""/>
+  <xacro:arg name="use_mock_hardware" default="true"/>
+  <xacro:arg name="include_hardware" default="true"/>
   <xacro:include filename="$(find za_description)/urdf/za_macro.xacro"/>
   <xacro:za_macro prefix="$(arg prefix)"/>
@@ -12,5 +14,7 @@
     <child link="$(arg prefix)base_link"/>
   </joint>
-  <xacro:include filename="$(find za_description)/urdf/za.ros2_control.xacro"/>
-  <xacro:za_ros2_control prefix="$(arg prefix)"/>
+  <xacro:if value="$(arg include_hardware)">
+    <xacro:include filename="$(find za_description)/urdf/za.ros2_control.xacro"/>
+    <xacro:za_ros2_control prefix="$(arg prefix)" use_mock_hardware="$(arg use_mock_hardware)"/>
+  </xacro:if>
 </robot>

Commit message: use config file for initial positions

File: urdf/za.ros2_control.xacro (robot description, xacro)
@@ -1,5 +1,11 @@
 <?xml version="1.0"?>
 <robot xmlns:xacro="http://www.ros.org/wiki/xacro">
-  <xacro:macro name="za_ros2_control" params="prefix use_mock_hardware:=^|true">
+  <xacro:macro name="za_ros2_control" params="
+    prefix
+    use_mock_hardware:=true
+    initial_positions_file:='$(find za_description)/config/initial_positions.yaml'">
+    <xacro:property
+      name="initial_positions"
+      value="${xacro.load_yaml(initial_positions_file)['initial_positions']}"/>
     <ros2_control name="${prefix}ros2_control" type="system">
       <hardware>
@@ -17,5 +23,5 @@
         </command_interface>
         <state_interface name="position">
-          <param name="initial_value">0.0</param>
+          <param name="initial_value">${initial_positions['joint_1']}</param>
         </state_interface>
         <state_interface name="velocity"/>
@@ -27,5 +33,5 @@
         </command_interface>
         <state_interface name="position">
-          <param name="initial_value">0.53</param>
+          <param name="initial_value">${initial_positions['joint_2']}</param>
         </state_interface>
         <state_interface name="velocity"/>
@@ -37,5 +43,5 @@
         </command_interface>
         <state_interface name="position">
-          <param name="initial_value">0.47</param>
+          <param name="initial_value">${initial_positions['joint_3']}</param>
         </state_interface>
         <state_interface name="velocity"/>
@@ -47,5 +53,5 @@
         </command_interface>
         <state_interface name="position">
-          <param name="initial_value">0.0</param>
+          <param name="initial_value">${initial_positions['joint_4']}</param>
         </state_interface>
         <state_interface name="velocity"/>
@@ -57,5 +63,5 @@
         </command_interface>
         <state_interface name="position">
-          <param name="initial_value">-1.0</param>
+          <param name="initial_value">${initial_positions['joint_5']}</param>
         </state_interface>
         <state_interface name="velocity"/>
@@ -67,5 +73,5 @@
         </command_interface>
         <state_interface name="position">
-          <param name="initial_value">0.0</param>
+          <param name="initial_value">${initial_positions['joint_6']}</param>
         </state_interface>
         <state_interface name="velocity"/>

File: urdf/za.xacro (robot description, xacro)
@@ -4,4 +4,6 @@
   <xacro:arg name="use_mock_hardware" default="true"/>
   <xacro:arg name="include_hardware" default="true"/>
+  <xacro:arg name="initial_positions_file"
+             default="$(find za_description)/config/initial_positions"/>
   <xacro:include filename="$(find za_description)/urdf/za_macro.xacro"/>
   <xacro:za_macro prefix="$(arg prefix)"/>
