Commit message: add 1 mm offsets back to links 3 and 5

File: urdf/za.xacro (robot description, xacro)
@@ -2,7 +2,6 @@
 <robot name="za" xmlns:xacro="http://www.ros.org/wiki/xacro">
   <xacro:arg name="prefix" default=""/>
-  <xacro:arg name="fixed_tool" default="True"/>
   <xacro:include filename="$(find za_description)/urdf/za_macro.xacro"/>
-  <xacro:za_macro prefix="$(arg prefix)" tool0_trans="0 0 0" tool0_rot="0 ${pi*1} 0" tool0_fixed="$(arg fixed_tool)"/>
+  <xacro:za_macro prefix="$(arg prefix)"/>
   <!-- 'world' frame: default pose reference frame -->
   <link name="world" />

File: urdf/za_macro.xacro (robot description, xacro)
@@ -127,5 +127,5 @@
     </joint>
     <joint name="${prefix}joint_3" type="revolute">
-      <origin rpy="0.0 0.0 0.0" xyz="0.0 0.0 0.454"/>
+      <origin rpy="0.0 0.0 0.0" xyz="0.0 -0.001 0.454"/>
       <axis xyz="0 1 0"/>
       <parent link="${prefix}link_2"/>
@@ -141,5 +141,5 @@
     </joint>
     <joint name="${prefix}joint_5" type="revolute">
-      <origin rpy="0.0 0.0 0.0" xyz="0.4195 0.0 0.0"/>
+      <origin rpy="0.0 0.0 0.0" xyz="0.4195 0.001 0.0"/>
       <axis xyz="0 1 0"/>
       <parent link="${prefix}link_4"/>

Commit message: add link inertias and gazebo transmissions

File: urdf/za.xacro (robot description, xacro)
@@ -12,3 +12,11 @@
     <child link="$(arg prefix)base_link"/>
   </joint>
+  <!-- Gazebo plugin for ROS Control -->
+  <gazebo>
+    <plugin name="gazebo_ros_control" filename="libgazebo_ros_control.so">
+      <controlPeriod>0.001</controlPeriod>
+      <robotSimType>za_gazebo/ZaHWSim</robotSimType>
+    </plugin>
+    <self_collide>true</self_collide>
+  </gazebo>
 </robot>

File: urdf/za_macro.xacro (robot description, xacro)
@@ -1,5 +1,8 @@
 <?xml version="1.0"?>
 <robot xmlns:xacro="http://www.ros.org/wiki/xacro">
+  <xacro:include filename="$(find za_description)/urdf/utils.xacro"/>"
   <xacro:macro name="za_macro" params="prefix">
+    <!-- Is the robot being simulated in gazebo?" -->
+    <xacro:arg name="gazebo" default="false" />
     <!-- link list -->
     <link name="${prefix}base_link">
@@ -14,4 +17,9 @@
         </geometry>
       </collision>
+      <inertial>
+        <origin xyz="-0.01236763 -0.00120116 0.13466856"/>
+        <mass value="18.32700000"/>
+        <inertia ixx="0.16366788" ixy="-0.00000166" ixz="-0.00348810" iyy="0.22044850" iyz="0.00000286" izz="0.17770306"/>
+      </inertial>
     </link>
     <link name="${prefix}link_1">
@@ -27,6 +35,7 @@
       </collision>
       <inertial>
-        <mass value="100"/>
-        <inertia ixx="1.0" ixy="0.0" ixz="0.0" iyy="1.0" iyz="0.0" izz="1.0"/>
+        <origin xyz="0.01021395 0.00697465 -0.07935107"/>
+        <mass value="13.44000000"/>
+        <inertia ixx="0.13591253" ixy="0.00009739" ixz="-0.00604284" iyy="0.11223931" iyz="0.00027520" izz="0.10172556"/>
       </inertial>
     </link>
@@ -43,6 +52,7 @@
       </collision>
       <inertial>
-        <mass value="100"/>
-        <inertia ixx="1.0" ixy="0.0" ixz="0.0" iyy="1.0" iyz="0.0" izz="1.0"/>
+        <origin xyz="-0.00387549 -0.00718854 0.27138897"/>
+        <mass value="17.11000000"/>
+        <inertia ixx="0.52527032" ixy="0.00015072" ixz="0.00040686" iyy="0.50042448" iyz="0.00016892" izz="0.09140527"/>
       </inertial>
     </link>
@@ -59,6 +69,7 @@
       </collision>
       <inertial>
-        <mass value="100"/>
-        <inertia ixx="1.0" ixy="0.0" ixz="0.0" iyy="1.0" iyz="0.0" izz="1.0"/>
+        <origin xyz="0.02825936 0.00083544 -0.00574226"/>
+        <mass value="7.33000000"/>
+        <inertia ixx="0.02513174" ixy="0.00012221" ixz="-0.00333856" iyy="0.03765338" iyz="-0.00009292" izz="0.02694824"/>
       </inertial>
     </link>
@@ -75,6 +86,7 @@
       </collision>
       <inertial>
-        <mass value="100"/>
-        <inertia ixx="1.0" ixy="0.0" ixz="0.0" iyy="1.0" iyz="0.0" izz="1.0"/>
+        <origin xyz="0.30544152 0.00346903 0.00392327"/>
+        <mass value="6.11000000"/>
+        <inertia ixx="0.01559502" ixy="-0.00031903" ixz="0.00008767" iyy="0.05602555" iyz="-0.00001324" izz="0.06119102"/>
       </inertial>
     </link>
@@ -91,6 +103,7 @@
       </collision>
       <inertial>
-        <mass value="100"/>
-        <inertia ixx="1.0" ixy="0.0" ixz="0.0" iyy="1.0" iyz="0.0" izz="1.0"/>
+        <origin xyz="-0.00517740 0.00016151 0.00015567"/>
+        <mass value="2.44000000"/>
+        <inertia ixx="0.00267434" ixy="0.00000003" ixz="-0.00000009" iyy="0.00582935" iyz="-0.00000003" izz="0.00571470"/>
       </inertial>
     </link>
@@ -107,6 +120,7 @@
       </collision>
       <inertial>
-        <mass value="100"/>
-        <inertia ixx="1.0" ixy="0.0" ixz="0.0" iyy="1.0" iyz="0.0" izz="1.0"/>
+        <origin xyz="-0.00968719 -0.00009104 0.00002796"/>
+        <mass value="0.24400000"/>
+        <inertia ixx="0.00010069" ixy="0.00000000" ixz="0.00000000" iyy="0.00006352" iyz="0.00000000" izz="0.00006352"/>
       </inertial>
     </link>
@@ -118,4 +132,5 @@
       <child link="${prefix}link_1"/>
       <limit effort="1000.0" lower="-2.96" upper="2.96" velocity="2.6"/>
+      <dynamics damping="0.003" friction="0.0" mu_coulomb="0" mu_viscous="16" />
     </joint>
     <joint name="${prefix}joint_2" type="revolute">
@@ -125,4 +140,5 @@
       <child link="${prefix}link_2"/>
       <limit effort="1000.0" lower="-1.74" upper="2.35" velocity="1.9"/>
+      <dynamics damping="0.003" friction="0.0" mu_coulomb="0" mu_viscous="16" />
     </joint>
     <joint name="${prefix}joint_3" type="revolute">
@@ -132,4 +148,5 @@
       <child link="${prefix}link_3"/>
       <limit effort="1000.0" lower="-1.570796" upper="1.15" velocity="2.6"/>
+      <dynamics damping="0.003" friction="0.0" mu_coulomb="0" mu_viscous="16" />
     </joint>
     <joint name="${prefix}joint_4" type="revolute">
@@ -139,4 +156,5 @@
       <child link="${prefix}link_4"/>
       <limit effort="1000.0" lower="-2.6" upper="2.6" velocity="3.5"/>
+      <dynamics damping="0.003" friction="0.0" mu_coulomb="0" mu_viscous="16" />
     </joint>
     <joint name="${prefix}joint_5" type="revolute">
@@ -146,4 +164,5 @@
       <child link="${prefix}link_5"/>
       <limit effort="1000.0" lower="-2.49" upper="2.49" velocity="3.9"/>
+      <dynamics damping="0.003" friction="0.0" mu_coulomb="0" mu_viscous="16" />
     </joint>
     <joint name="${prefix}joint_6" type="revolute">
@@ -153,4 +172,5 @@
       <child link="${prefix}link_6"/>
       <limit effort="1000.0" lower="${pi*-1}" upper="${pi*1}" velocity="${pi*2}"/>
+      <dynamics damping="0.003" friction="0.0" mu_coulomb="0" mu_viscous="16" />
     </joint>
     <!-- ROS-Industrial 'base' frame: base_link to Fanuc World Coordinates transform -->
@@ -176,4 +196,30 @@
       <child link="${prefix}tool0" />
     </joint>
+    <!-- Define additional Gazebo tags -->
+    <xacro:if value="$(arg gazebo)">
+      <xacro:gazebo-joint joint="${prefix}joint_1" transmission="hardware_interface/EffortJointInterface" />
+      <xacro:gazebo-joint joint="${prefix}joint_2" transmission="hardware_interface/EffortJointInterface" />
+      <xacro:gazebo-joint joint="${prefix}joint_3" transmission="hardware_interface/EffortJointInterface" />
+      <xacro:gazebo-joint joint="${prefix}joint_4" transmission="hardware_interface/EffortJointInterface" />
+      <xacro:gazebo-joint joint="${prefix}joint_5" transmission="hardware_interface/EffortJointInterface" />
+      <xacro:gazebo-joint joint="${prefix}joint_6" transmission="hardware_interface/EffortJointInterface" />
+      <xacro:gazebo-joint joint="${prefix}joint_1" transmission="hardware_interface/VelocityJointInterface" />
+      <xacro:gazebo-joint joint="${prefix}joint_2" transmission="hardware_interface/VelocityJointInterface" />
+      <xacro:gazebo-joint joint="${prefix}joint_3" transmission="hardware_interface/VelocityJointInterface" />
+      <xacro:gazebo-joint joint="${prefix}joint_4" transmission="hardware_interface/VelocityJointInterface" />
+      <xacro:gazebo-joint joint="${prefix}joint_5" transmission="hardware_interface/VelocityJointInterface" />
+      <xacro:gazebo-joint joint="${prefix}joint_6" transmission="hardware_interface/VelocityJointInterface" />
+      <xacro:gazebo-joint joint="${prefix}joint_1" transmission="hardware_interface/PositionJointInterface" />
+      <xacro:gazebo-joint joint="${prefix}joint_2" transmission="hardware_interface/PositionJointInterface" />
+      <xacro:gazebo-joint joint="${prefix}joint_3" transmission="hardware_interface/PositionJointInterface" />
+      <xacro:gazebo-joint joint="${prefix}joint_4" transmission="hardware_interface/PositionJointInterface" />
+      <xacro:gazebo-joint joint="${prefix}joint_5" transmission="hardware_interface/PositionJointInterface" />
+      <xacro:gazebo-joint joint="${prefix}joint_6" transmission="hardware_interface/PositionJointInterface" />
+      <xacro:transmission-za-state arm_id="${prefix}" />
+      <xacro:transmission-za-model arm_id="${prefix}"
+         root="${prefix}joint_1"
+         tip="${prefix}joint_6-flange"
+      />
+    </xacro:if>
   </xacro:macro>
 </robot>

Commit message: remove Gazebo tags and update joint limits
Joint limits were measured on the physical robot

File: urdf/za.xacro (robot description, xacro)
@@ -8,15 +8,6 @@
   <joint name="world-$(arg prefix)base_link" type="fixed">
     <origin xyz="0 0 0" rpy="0 0 0"/>
-    <axis xyz="0 0 1"/>
     <parent link="world"/>
     <child link="$(arg prefix)base_link"/>
   </joint>
-  <!-- Gazebo plugin for ROS Control -->
-  <gazebo>
-    <plugin name="gazebo_ros_control" filename="libgazebo_ros_control.so">
-      <controlPeriod>0.001</controlPeriod>
-      <robotSimType>za_gazebo/ZaHWSim</robotSimType>
-    </plugin>
-    <self_collide>true</self_collide>
-  </gazebo>
 </robot>

File: urdf/za_macro.xacro (robot description, xacro)
@@ -1,8 +1,5 @@
 <?xml version="1.0"?>
 <robot xmlns:xacro="http://www.ros.org/wiki/xacro">
-  <xacro:include filename="$(find za_description)/urdf/utils.xacro"/>"
   <xacro:macro name="za_macro" params="prefix">
-    <!-- Is the robot being simulated in gazebo?" -->
-    <xacro:arg name="gazebo" default="true" />
     <!-- link list -->
     <link name="${prefix}base_link">
@@ -17,9 +14,4 @@
         </geometry>
       </collision>
-      <inertial>
-        <origin xyz="-0.035356 -0.000003 0.142049"/>
-        <mass value="18.327"/>
-        <inertia ixx="0.185203" ixy="0.000006" ixz="0.016506" iyy="0.232301" iyz="0.000014" izz="0.163415"/>
-      </inertial>
     </link>
     <link name="${prefix}link_1">
@@ -34,9 +26,4 @@
         </geometry>
       </collision>
-      <inertial>
-        <origin xyz="0.009612 0.016390 -0.065742"/>
-        <mass value="13.44"/>
-        <inertia ixx="0.178493" ixy="0.002772" ixz="0.010363" iyy="0.126756" iyz="0.016161" izz="0.130031"/>
-      </inertial>
     </link>
     <link name="${prefix}link_2">
@@ -51,9 +38,4 @@
         </geometry>
       </collision>
-      <inertial>
-        <origin xyz="-0.003803 0.001296 0.191397"/>
-        <mass value="17.11"/>
-        <inertia ixx="0.740919" ixy="-0.003160" ixz="-0.003160" iyy="0.699365" iyz="0.039435" izz="0.100361"/>
-      </inertial>
     </link>
     <link name="${prefix}link_3">
@@ -68,9 +50,4 @@
         </geometry>
       </collision>
-      <inertial>
-        <origin xyz="0.019381 -0.007200 -0.002694"/>
-        <mass value="7.33"/>
-        <inertia ixx="0.027465" ixy="0.001126" ixz="0.004749" iyy="0.037555" iyz="-0.000148" izz="0.031377"/>
-      </inertial>
     </link>
     <link name="${prefix}link_4">
@@ -85,9 +62,4 @@
         </geometry>
       </collision>
-      <inertial>
-        <origin xyz="0.290062 0.005593 0.000640"/>
-        <mass value="6.11"/>
-        <inertia ixx="0.019909" ixy="0.003159" ixz="-0.000103" iyy="0.058941" iyz="-0.000022" izz="0.066959"/>
-      </inertial>
     </link>
     <link name="${prefix}link_5">
@@ -102,9 +74,4 @@
         </geometry>
       </collision>
-      <inertial>
-        <origin xyz="0.009621 0.000953 0.000305"/>
-        <mass value="2.44"/>
-        <inertia ixx="0.002635" ixy="-0.000031" ixz="-0.000023" iyy="0.005551" iyz="0.000004" izz="0.005487"/>
-      </inertial>
     </link>
     <link name="${prefix}link_6">
@@ -119,64 +86,52 @@
         </geometry>
       </collision>
-      <inertial>
-        <origin xyz="-0.012049 0.000000 0.000000"/>
-        <mass value="0.244"/>
-        <inertia ixx="0.000106" ixy="0.000000" ixz="0.000000" iyy="0.000064" iyz="0.000000" izz="0.000064"/>
-      </inertial>
     </link>
     <!-- joint list -->
     <joint name="${prefix}joint_1" type="revolute">
+      <parent link="${prefix}base_link"/>
+      <child link="${prefix}link_1"/>
       <origin rpy="0.0 0.0 0.0" xyz="0 0 0.45"/>
       <axis xyz="0 0 1"/>
-      <parent link="${prefix}base_link"/>
-      <child link="${prefix}link_1"/>
-      <limit effort="500.0" lower="-2.96" upper="2.96" velocity="2.6"/>
-      <dynamics damping="0.003" friction="0.0"/>
-  </joint>
+      <limit effort="0" lower="${radians(-170)}" upper="${radians(170)}" velocity="${radians(150)}"/>
+    </joint>
     <joint name="${prefix}joint_2" type="revolute">
+      <parent link="${prefix}link_1"/>
+      <child link="${prefix}link_2"/>
       <origin rpy="0.0 0.0 0.0" xyz="0.025 0 0.0"/>
       <axis xyz="0 1 0"/>
-      <parent link="${prefix}link_1"/>
-      <child link="${prefix}link_2"/>
-      <limit effort="500.0" lower="-1.74" upper="2.35" velocity="1.9"/>
-      <dynamics damping="0.003" friction="0.0"/>
+      <limit effort="0" lower="${radians(-100)}" upper="${radians(130)}" velocity="${radians(112.5)}"/>
     </joint>
     <joint name="${prefix}joint_3" type="revolute">
+      <parent link="${prefix}link_2"/>
+      <child link="${prefix}link_3"/>
       <origin rpy="0.0 0.0 0.0" xyz="0.0 -0.001 0.454"/>
       <axis xyz="0 1 0"/>
-      <parent link="${prefix}link_2"/>
-      <child link="${prefix}link_3"/>
-      <limit effort="200.0" lower="-1.570796" upper="1.15" velocity="2.6"/>
-      <dynamics damping="0.003" friction="0.0"/>
+      <limit effort="0" lower="${radians(-120)}" upper="${radians(65)}" velocity="${radians(150)}"/>
     </joint>
     <joint name="${prefix}joint_4" type="revolute">
+      <parent link="${prefix}link_3"/>
+      <child link="${prefix}link_4"/>
       <origin rpy="0.0 0.0 0.0" xyz="0.0 0.0 0.035"/>
       <axis xyz="1 0 0"/>
-      <parent link="${prefix}link_3"/>
-      <child link="${prefix}link_4"/>
-      <limit effort="100.0" lower="-2.6" upper="2.6" velocity="3.5"/>
-      <dynamics damping="0.003" friction="0.0"/>
+      <limit effort="0" lower="${radians(-180)}" upper="${radians(180)}" velocity="${radians(204.5)}"/>
     </joint>
     <joint name="${prefix}joint_5" type="revolute">
+      <parent link="${prefix}link_4"/>
+      <child link="${prefix}link_5"/>
       <origin rpy="0.0 0.0 0.0" xyz="0.4195 0.001 0.0"/>
       <axis xyz="0 1 0"/>
-      <parent link="${prefix}link_4"/>
-      <child link="${prefix}link_5"/>
-      <limit effort="100.0" lower="-2.49" upper="2.49" velocity="3.9"/>
-      <dynamics damping="0.003" friction="0.0"/>
+      <limit effort="0" lower="${radians(-140)}" upper="${radians(140)}" velocity="${radians(225)}"/>
     </joint>
     <joint name="${prefix}joint_6" type="revolute">
+      <parent link="${prefix}link_5"/>
+      <child link="${prefix}link_6"/>
       <origin rpy="0.0 0.0 0.0" xyz="0.1175 0.0 0.0"/>
       <axis xyz="1 0 0"/>
-      <parent link="${prefix}link_5"/>
-      <child link="${prefix}link_6"/>
-      <limit effort="10.0" lower="${pi*-1}" upper="${pi*1}" velocity="${pi*2}"/>
-      <dynamics damping="0.003" friction="0.0"/>
+      <limit effort="0" lower="${radians(-360)}" upper="${radians(360)}" velocity="${radians(360)}"/>
     </joint>
-    <!-- ROS-Industrial 'base' frame: base_link to Fanuc World Coordinates transform -->
+    <!-- ROS-Industrial 'base' frame: base_link to Tormach World Coordinates transform -->
     <link name="${prefix}base" />
     <joint name="${prefix}base_link-base" type="fixed">
       <origin xyz="0 0 0" rpy="0 0 0"/>
-      <axis xyz="0 0 1"/>
       <parent link="${prefix}base_link"/>
       <child link="${prefix}base"/>
@@ -185,41 +140,15 @@
     <link name="${prefix}flange" />
     <joint name="${prefix}joint_6-flange" type="fixed">
-      <origin xyz="0 0 0" rpy="0 0 0" />
-      <parent link="${prefix}link_6" />
-      <child link="${prefix}flange" />
+      <origin xyz="0 0 0" rpy="0 0 0"/>
+      <parent link="${prefix}link_6"/>
+      <child link="${prefix}flange"/>
     </joint>
     <!-- ROS-Industrial 'tool0' frame: all-zeros tool frame -->
     <link name="${prefix}tool0" />
-    <joint name="${prefix}link_6_tool0" type="fixed">
-      <origin xyz="0 0 0" rpy="0 ${pi/2} 0" />
-      <parent link="${prefix}flange" />
-      <child link="${prefix}tool0" />
+    <joint name="${prefix}link_6-tool0" type="fixed">
+      <origin xyz="0 0 0" rpy="0 ${pi/2} 0"/>
+      <parent link="${prefix}flange"/>
+      <child link="${prefix}tool0"/>
     </joint>
-    <!-- Define additional Gazebo tags -->
-    <xacro:if value="$(arg gazebo)">
-      <xacro:gazebo-joint joint="${prefix}joint_1" transmission="hardware_interface/EffortJointInterface" reduction="1.5"/>
-      <xacro:gazebo-joint joint="${prefix}joint_2" transmission="hardware_interface/EffortJointInterface" reduction="100"/>
-      <xacro:gazebo-joint joint="${prefix}joint_3" transmission="hardware_interface/EffortJointInterface" reduction="50"/>
-      <xacro:gazebo-joint joint="${prefix}joint_4" transmission="hardware_interface/EffortJointInterface" reduction="1.25"/>
-      <xacro:gazebo-joint joint="${prefix}joint_5" transmission="hardware_interface/EffortJointInterface" reduction="50"/>
-      <xacro:gazebo-joint joint="${prefix}joint_6" transmission="hardware_interface/EffortJointInterface" reduction="30"/>
-      <xacro:gazebo-joint joint="${prefix}joint_1" transmission="hardware_interface/VelocityJointInterface" reduction="1.5"/>
-      <xacro:gazebo-joint joint="${prefix}joint_2" transmission="hardware_interface/VelocityJointInterface" reduction="100"/>
-      <xacro:gazebo-joint joint="${prefix}joint_3" transmission="hardware_interface/VelocityJointInterface" reduction="50"/>
-      <xacro:gazebo-joint joint="${prefix}joint_4" transmission="hardware_interface/VelocityJointInterface" reduction="1.25"/>
-      <xacro:gazebo-joint joint="${prefix}joint_5" transmission="hardware_interface/VelocityJointInterface" reduction="50"/>
-      <xacro:gazebo-joint joint="${prefix}joint_6" transmission="hardware_interface/VelocityJointInterface" reduction="30"/>
-      <xacro:gazebo-joint joint="${prefix}joint_1" transmission="hardware_interface/PositionJointInterface" reduction="1.5"/>
-      <xacro:gazebo-joint joint="${prefix}joint_2" transmission="hardware_interface/PositionJointInterface" reduction="100"/>
-      <xacro:gazebo-joint joint="${prefix}joint_3" transmission="hardware_interface/PositionJointInterface" reduction="50"/>
-      <xacro:gazebo-joint joint="${prefix}joint_4" transmission="hardware_interface/PositionJointInterface" reduction="1.25"/>
-      <xacro:gazebo-joint joint="${prefix}joint_5" transmission="hardware_interface/PositionJointInterface" reduction="50"/>
-      <xacro:gazebo-joint joint="${prefix}joint_6" transmission="hardware_interface/PositionJointInterface" reduction="30"/>
-      <xacro:transmission-za-state arm_id="${prefix}" />
-      <xacro:transmission-za-model arm_id="${prefix}"
-         root="${prefix}joint_1"
-         tip="${prefix}joint_6-flange"
-      />
-    </xacro:if>
   </xacro:macro>
 </robot>
