Commit message: define joint limits with yaml

File: urdf/za.xacro (robot description, xacro)
@@ -5,7 +5,9 @@
   <xacro:arg name="include_hardware" default="true"/>
   <xacro:arg name="initial_positions_file"
-             default="$(find za_description)/config/initial_positions"/>
+    default="$(find za_description)/config/initial_positions.yaml"/>
+  <xacro:arg name="joint_limits_file"
+    default="$(find za_description)/config/joint_limits.yaml"/>
   <xacro:include filename="$(find za_description)/urdf/za_macro.xacro"/>
-  <xacro:za_macro prefix="$(arg prefix)"/>
+  <xacro:za_macro prefix="$(arg prefix)" joint_limits_parameters_file="$(arg joint_limits_file)"/>
   <!-- 'world' frame - default pose reference frame -->
   <link name="world" />

File: urdf/za_macro.xacro (robot description, xacro)
@@ -1,5 +1,10 @@
 <?xml version="1.0"?>
 <robot xmlns:xacro="http://www.ros.org/wiki/xacro">
-  <xacro:macro name="za_macro" params="prefix">
+  <xacro:macro name="za_macro" params="
+    prefix
+    joint_limits_parameters_file
+    ">
+  <xacro:property name="joint_limits_parameters" value="${xacro.load_yaml(joint_limits_parameters_file)}"/>
+  <xacro:property name="joint_limits" value="${joint_limits_parameters['joint_limits']}"/>
     <!-- link list -->
     <link name="${prefix}base_link">
@@ -93,5 +98,9 @@
       <origin rpy="0.0 0.0 0.0" xyz="0 0 0.45"/>
       <axis xyz="0 0 1"/>
-      <limit effort="0" lower="${radians(-170)}" upper="${radians(170)}" velocity="${radians(150)}"/>
+      <limit
+        effort="${joint_limits['joint_1']['max_effort']}"
+        lower="${joint_limits['joint_1']['min_position']}"
+        upper="${joint_limits['joint_1']['max_position']}"
+        velocity="${joint_limits['joint_1']['max_velocity']}"/>
     </joint>
     <joint name="${prefix}joint_2" type="revolute">
@@ -100,5 +109,9 @@
       <origin rpy="0.0 0.0 0.0" xyz="0.025 0 0.0"/>
       <axis xyz="0 1 0"/>
-      <limit effort="0" lower="${radians(-100)}" upper="${radians(130)}" velocity="${radians(112.5)}"/>
+      <limit
+        effort="${joint_limits['joint_2']['max_effort']}"
+        lower="${joint_limits['joint_2']['min_position']}"
+        upper="${joint_limits['joint_2']['max_position']}"
+        velocity="${joint_limits['joint_2']['max_velocity']}"/>
     </joint>
     <joint name="${prefix}joint_3" type="revolute">
@@ -107,5 +120,9 @@
       <origin rpy="0.0 0.0 0.0" xyz="0.0 -0.001 0.454"/>
       <axis xyz="0 1 0"/>
-      <limit effort="0" lower="${radians(-120)}" upper="${radians(65)}" velocity="${radians(150)}"/>
+      <limit
+        effort="${joint_limits['joint_3']['max_effort']}"
+        lower="${joint_limits['joint_3']['min_position']}"
+        upper="${joint_limits['joint_3']['max_position']}"
+        velocity="${joint_limits['joint_3']['max_velocity']}"/>
     </joint>
     <joint name="${prefix}joint_4" type="revolute">
@@ -114,5 +131,9 @@
       <origin rpy="0.0 0.0 0.0" xyz="0.0 0.0 0.035"/>
       <axis xyz="1 0 0"/>
-      <limit effort="0" lower="${radians(-180)}" upper="${radians(180)}" velocity="${radians(204.5)}"/>
+      <limit
+        effort="${joint_limits['joint_4']['max_effort']}"
+        lower="${joint_limits['joint_4']['min_position']}"
+        upper="${joint_limits['joint_4']['max_position']}"
+        velocity="${joint_limits['joint_4']['max_velocity']}"/>
     </joint>
     <joint name="${prefix}joint_5" type="revolute">
@@ -121,5 +142,9 @@
       <origin rpy="0.0 0.0 0.0" xyz="0.4195 0.001 0.0"/>
       <axis xyz="0 1 0"/>
-      <limit effort="0" lower="${radians(-140)}" upper="${radians(140)}" velocity="${radians(225)}"/>
+      <limit
+        effort="${joint_limits['joint_5']['max_effort']}"
+        lower="${joint_limits['joint_5']['min_position']}"
+        upper="${joint_limits['joint_5']['max_position']}"
+        velocity="${joint_limits['joint_5']['max_velocity']}"/>
     </joint>
     <joint name="${prefix}joint_6" type="revolute">
@@ -128,5 +153,9 @@
       <origin rpy="0.0 0.0 0.0" xyz="0.1175 0.0 0.0"/>
       <axis xyz="1 0 0"/>
-      <limit effort="0" lower="${radians(-360)}" upper="${radians(360)}" velocity="${radians(360)}"/>
+      <limit
+        effort="${joint_limits['joint_6']['max_effort']}"
+        lower="${joint_limits['joint_6']['min_position']}"
+        upper="${joint_limits['joint_6']['max_position']}"
+        velocity="${joint_limits['joint_6']['max_velocity']}"/>
     </joint>
     <!-- ROS-Industrial 'base' frame - base_link to Tormach World Coordinates transform -->
